File: MultiUse_Battery/MultiUse_Battery.kicad_pcb (KiCad board)
At the start: 2 copper layers, 50 x 30 mm, 14 parts, among them IC1 ATMEGA328P-AU, P3 CONN_01X03, P4 CONN_01X03, P5 CONN_02X03, P6 CONN_01X02, U1 MAX1724, U3 RFM69HW

Commit message: Ajout README.md Modification orientation support pile CR2032 Ajout d'une PULLUP sur 2eme entrée
Parts:
- added R2: 4K7, Resistors_SMD:R_1206_HandSoldering, F.Cu at (100.7, 58.3)
- moved 3V3 22.8 mm to (89.2, 67.8), turned to 0 degrees
- moved R1 0.13 mm to (86.4, 58.3)
Routing:
- net /VIN: track 67.8 -> 53.0 mm
- net /3V3: track 130.7 -> 135.2 mm
- net /GND: track 42.5 -> 44.1 mm
- net /PC1: track 9.85 -> 11.2 mm
- net (no net): track 0.00 -> 0.74 mm
Changed lines of the file:
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@@
 (kicad_pcb (version 4) (host pcbnew 4.0.5-e0-6337~49~ubuntu16.04.1)
   (general
-    (links 43)
+    (links 45)
     (no_connects 0)
     (area 81.547999 51.862999 131.698001 82.013001)
     (thickness 1.6)
     (drawings 5)
-    (tracks 181)
+    (tracks 190)
     (zones 0)
-    (modules 14)
+    (modules 15)
     (nets 38)
   )
@@
   )
   (module Resistors_SMD:R_1206_HandSoldering (layer F.Cu)
-    (at 86.36 58.42)
+    (at 86.36 58.293)
     (descr "Resistor SMD 1206, hand soldering")
     (tags "resistor 1206")
@@
   )
   (module Batteries:BU2032_smd (layer B.Cu)
-    (at 110.109 76.708 145)
-    (fp_text reference 3V3 (at 0.863015 -3.860095 145) (layer B.SilkS)
+    (at 89.154 67.818)
+    (fp_text reference 3V3 (at 0.863015 -3.860095) (layer B.SilkS)
       (effects (font (size 1 1) (thickness 0.15)) (justify mirror))
     )
-    (fp_text value CONN_01X02 (at 14 -2 145) (layer B.SilkS)
+    (fp_text value CONN_01X02 (at 14 -2) (layer B.SilkS)
       (effects (font (size 1 1) (thickness 0.15)) (justify mirror))
     )
@@
     (fp_line (start -2.5 3) (end -2.5 -3) (layer B.SilkS) (width 0.15))
     (fp_line (start -2.5 -3) (end 4.5 -3) (layer B.SilkS) (width 0.15))
-    (pad 2 smd rect (at 29.3 0 145) (size 5 4.2) (layers B.Cu B.Paste B.Mask)
-      (net 1 /GND))
-    (pad 1 smd rect (at 0 0 145) (size 5 4.2) (layers B.Cu B.Paste B.Mask)
+    (pad 2 smd rect (at 29.3 0) (size 5 4.2) (layers B.Cu B.Paste B.Mask)
+      (net 1 /GND))
+    (pad 1 smd rect (at 0 0) (size 5 4.2) (layers B.Cu B.Paste B.Mask)
       (net 36 /VIN))
   )
@@
     )
   )
+  (module Resistors_SMD:R_1206_HandSoldering (layer F.Cu)
+    (at 100.711 58.293)
+    (descr "Resistor SMD 1206, hand soldering")
+    (tags "resistor 1206")
+    (attr smd)
+    (fp_text reference R2 (at 0 -2.3) (layer F.SilkS)
+      (effects (font (size 1 1) (thickness 0.15)))
+    )
+    (fp_text value 4K7 (at 0 2.3) (layer F.Fab)
+      (effects (font (size 1 1) (thickness 0.15)))
+    )
+    (fp_line (start -1.6 0.8) (end -1.6 -0.8) (layer F.Fab) (width 0.1))
+    (fp_line (start 1.6 0.8) (end -1.6 0.8) (layer F.Fab) (width 0.1))
+    (fp_line (start 1.6 -0.8) (end 1.6 0.8) (layer F.Fab) (width 0.1))
+    (fp_line (start -1.6 -0.8) (end 1.6 -0.8) (layer F.Fab) (width 0.1))
+    (fp_line (start -3.3 -1.2) (end 3.3 -1.2) (layer F.CrtYd) (width 0.05))
+    (fp_line (start -3.3 1.2) (end 3.3 1.2) (layer F.CrtYd) (width 0.05))
+    (fp_line (start -3.3 -1.2) (end -3.3 1.2) (layer F.CrtYd) (width 0.05))
+    (fp_line (start 3.3 -1.2) (end 3.3 1.2) (layer F.CrtYd) (width 0.05))
+    (fp_line (start 1 1.075) (end -1 1.075) (layer F.SilkS) (width 0.15))
+    (fp_line (start -1 -1.075) (end 1 -1.075) (layer F.SilkS) (width 0.15))
+    (pad 1 smd rect (at -2 0) (size 2 1.7) (layers F.Cu F.Paste F.Mask)
+      (net 2 /3V3))
+    (pad 2 smd rect (at 2 0) (size 2 1.7) (layers F.Cu F.Paste F.Mask)
+      (net 21 /PC1))
+    (model Resistors_SMD.3dshapes/R_1206_HandSoldering.wrl
+      (at (xyz 0 0 0))
+      (scale (xyz 1 1 1))
+      (rotate (xyz 0 0 0))
+    )
+  )
   (gr_line (start 131.623 81.938) (end 131.623 51.938) (angle 90) (layer Edge.Cuts) (width 0.15))
   (gr_line (start 81.623 81.938) (end 131.623 81.938) (angle 90) (layer Edge.Cuts) (width 0.15))
@@
   (gr_line (start 131.623 51.938) (end 81.623 51.938) (angle 90) (layer Edge.Cuts) (width 0.15))
   (gr_line (start 81.623 51.938) (end 131.623 51.938) (angle 90) (layer Edge.Cuts) (width 0.15))
+  (segment (start 110.109 76.708) (end 110.109 77.089) (width 0.25) (layer B.Cu) (net 0))
+  (segment (start 109.855 76.962) (end 110.109 76.708) (width 0.25) (layer B.Cu) (net 0))
+  (segment (start 99.295 62.171) (end 99.295 61.233) (width 0.25) (layer F.Cu) (net 1))
+  (segment (start 99.295 61.233) (end 100.584 59.944) (width 0.25) (layer F.Cu) (net 1))
+  (segment (start 105.2703 58.5597) (end 105.2703 54.4322) (width 0.25) (layer F.Cu) (net 1))
+  (segment (start 103.886 59.944) (end 105.2703 58.5597) (width 0.25) (layer F.Cu) (net 1))
+  (segment (start 100.584 59.944) (end 103.886 59.944) (width 0.25) (layer F.Cu) (net 1))
   (segment (start 87.4903 75.04176) (end 87.4903 73.4187) (width 0.25) (layer F.Cu) (net 1))
   (segment (start 93.123 79.089) (end 91.44 79.089) (width 0.25) (layer F.Cu) (net 1))
@@
   (segment (start 100.095 72.244) (end 99.949 72.39) (width 0.25) (layer F.Cu) (net 1))
   (segment (start 99.949 72.39) (end 99.822 72.517) (width 0.25) (layer F.Cu) (net 1))
-  (segment (start 99.295 62.171) (end 99.295 61.233) (width 0.25) (layer F.Cu) (net 1))
-  (segment (start 99.295 61.233) (end 103.759 56.769) (width 0.25) (layer F.Cu) (net 1))
-  (segment (start 103.759 56.769) (end 104.267 56.769) (width 0.25) (layer F.Cu) (net 1))
-  (segment (start 104.267 56.769) (end 105.2703 55.7657) (width 0.25) (layer F.Cu) (net 1))
-  (segment (start 105.2703 55.7657) (end 105.2703 54.4322) (width 0.25) (layer F.Cu) (net 1))
+  (segment (start 98.711 58.293) (end 98.711 55.9115) (width 0.25) (layer F.Cu) (net 2))
+  (segment (start 98.711 55.9115) (end 100.1903 54.4322) (width 0.25) (layer F.Cu) (net 2))
   (segment (start 90.678 69.437) (end 90.678 71.44004) (width 0.25) (layer F.Cu) (net 2))
   (segment (start 90.678 71.44004) (end 90.678 71.374) (width 0.25) (layer F.Cu) (net 2))
@@
   (segment (start 127.6985 54.6608) (end 127.6985 59.2985) (width 0.25) (layer F.Cu) (net 19))
   (segment (start 127.6985 59.2985) (end 127.7224 59.3224) (width 0.25) (layer F.Cu) (net 19))
+  (segment (start 127.6985 59.2985) (end 127.7224 59.3224) (width 0.25) (layer F.Cu) (net 19))
   (segment (start 127.443 54.294) (end 127.508 54.229) (width 0.25) (layer F.Cu) (net 19))
   (segment (start 86.7029 56.7629) (end 88.36 58.42) (width 0.25) (layer F.Cu) (net 20))
@@
   (segment (start 96.895 62.171) (end 96.842 62.171) (width 0.25) (layer F.Cu) (net 20))
   (segment (start 96.842 62.171) (end 93.091 58.42) (width 0.25) (layer F.Cu) (net 20))
-  (segment (start 102.7303 54.4322) (end 102.7303 55.2577) (width 0.25) (layer F.Cu) (net 21))
-  (segment (start 102.7303 55.2577) (end 97.663 60.325) (width 0.25) (layer F.Cu) (net 21))
-  (segment (start 97.663 60.325) (end 97.663 62.139) (width 0.25) (layer F.Cu) (net 21))
+  (segment (start 97.695 62.171) (end 97.695 61.309) (width 0.25) (layer F.Cu) (net 21))
+  (segment (start 98.933 60.071) (end 99.441 60.071) (width 0.25) (layer F.Cu) (net 21))
+  (segment (start 97.695 61.309) (end 98.933 60.071) (width 0.25) (layer F.Cu) (net 21))
+  (segment (start 102.711 58.293) (end 101.346 58.293) (width 0.25) (layer F.Cu) (net 21))
+  (segment (start 101.346 58.293) (end 99.568 60.071) (width 0.25) (layer F.Cu) (net 21))
+  (segment (start 99.568 60.071) (end 99.441 60.071) (width 0.25) (layer F.Cu) (net 21))
+  (segment (start 102.7303 54.4322) (end 102.7303 58.2737) (width 0.25) (layer F.Cu) (net 21))
+  (segment (start 102.7303 58.2737) (end 102.711 58.293) (width 0.25) (layer F.Cu) (net 21))
+  (segment (start 102.584 54.5785) (end 102.7303 54.4322) (width 0.25) (layer F.Cu) (net 21))
   (segment (start 97.663 62.139) (end 97.695 62.171) (width 0.25) (layer F.Cu) (net 21))
   (segment (start 108.585 63.627) (end 109.093 63.627) (width 0.25) (layer F.Cu) (net 22))
@@
   (via (at 114.554 64.135) (size 0.6) (drill 0.4) (layers F.Cu B.Cu) (net 28))
   (segment (start 117.7224 60.9666) (end 114.554 64.135) (width 0.25) (layer F.Cu) (net 28))
+  (segment (start 89.154 67.818) (end 89.154 71.628) (width 0.25) (layer B.Cu) (net 36) (status 400000))
+  (segment (start 84.455 76.327) (end 84.455 79.629) (width 0.25) (layer B.Cu) (net 36) (status 800000))
+  (segment (start 89.154 71.628) (end 84.455 76.327) (width 0.25) (layer B.Cu) (net 36))
   (segment (start 88.138 77.089) (end 85.98916 77.089) (width 0.25) (layer F.Cu) (net 36))
   (segment (start 85.98916 77.089) (end 85.9155 77.01534) (width 0.25) (layer F.Cu) (net 36))
@@
   (segment (start 85.09 67.437) (end 82.804 69.723) (width 0.25) (layer F.Cu) (net 36))
   (segment (start 84.455 79.629) (end 84.455 80.264) (width 0.25) (layer B.Cu) (net 36))
-  (segment (start 84.455 80.264) (end 85.344 81.153) (width 0.25) (layer B.Cu) (net 36))
-  (segment (start 105.664 81.153) (end 110.109 76.708) (width 0.25) (layer B.Cu) (net 36))
-  (segment (start 85.344 81.153) (end 105.664 81.153) (width 0.25) (layer B.Cu) (net 36))
-  (segment (start 110.109 76.708) (end 110.109 77.089) (width 0.25) (layer B.Cu) (net 36))
-  (segment (start 109.855 76.962) (end 110.109 76.708) (width 0.25) (layer B.Cu) (net 36))
   (segment (start 84.4423 75.54214) (end 84.4423 79.6163) (width 0.25) (layer F.Cu) (net 36))
   (segment (start 84.4423 79.6163) (end 84.455 79.629) (width 0.25) (layer F.Cu) (net 36))

Commit message: modifs
Parts:
- added U2: AP111733, TO_SOT_Packages_SMD:SOT-223, F.Cu at (87.6, 63.6)
- moved C2 2.82 mm to (92.3, 69.7)
Routing:
- net /3V3: track 135.2 -> 164.5 mm, vias 1 -> 0
- net /GND: track 44.1 -> 59.9 mm, vias 0 -> 1
- net /VIN: track 53.0 -> 57.4 mm
- net /SCK: track 28.3 -> 29.8 mm
- net (no net): track 0.74 -> 0.00 mm

Commit message: Ajout GERBER
Parts:
- 3V3: value CONN_01X02 -> CR2032
- renumbered C1 to 10uF, C2 to 10uF, U2 to 1117, IC1 to 328p, P6 to 3V3, R1 to 4K7, R2 to 4K7, P5 to ICSP, U3 to RFM69HW, P3 to S0, P4 to S1, 3V3 to VIN
Changed lines of the file:
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@@
     (links 49)
     (no_connects 0)
-    (area 81.547999 51.862999 131.698001 82.013001)
+    (area 81.547999 51.476 131.779334 82.355)
     (thickness 1.6)
     (drawings 5)
@@
   (page A4)
   (layers
-    (0 F.Cu signal)
-    (31 B.Cu signal)
+    (0 F.Cu signal hide)
+    (31 B.Cu signal hide)
     (32 B.Adhes user)
     (33 F.Adhes user)
@@
     (47 F.CrtYd user)
     (48 B.Fab user)
-    (49 F.Fab user)
+    (49 F.Fab user hide)
   )
   (setup
@@
     (mod_text_size 1 1)
     (mod_text_width 0.15)
-    (pad_size 1.524 1.524)
-    (pad_drill 0.762)
+    (pad_size 1.7272 1.7272)
+    (pad_drill 0.3)
     (pad_to_mask_clearance 0.2)
     (aux_axis_origin 0 0)
     (visible_elements 7FFFFFFF)
     (pcbplotparams
-      (layerselection 0x00030_80000001)
-      (usegerberextensions false)
+      (layerselection 0x010f0_80000001)
+      (usegerberextensions true)
       (excludeedgelayer true)
       (linewidth 0.100000)
@@
       (outputformat 1)
       (mirror false)
-      (drillshape 1)
+      (drillshape 0)
       (scaleselection 1)
-      (outputdirectory ""))
+      (outputdirectory GERBER/))
   )
   (net 0 "")
@@
     (tags "capacitor 1206")
     (attr smd)
-    (fp_text reference C1 (at 0 -2.3 270) (layer F.SilkS)
+    (fp_text reference 10uF (at 0 -1.905 270) (layer F.SilkS)
       (effects (font (size 1 1) (thickness 0.15)))
     )
@@
     (descr RFM69HW)
     (tags "RFM69HW, RF69")
-    (fp_text reference U3 (at 0.254 -1.778 90) (layer F.SilkS)
+    (fp_text reference RFM69HW (at 0.254 -1.778 90) (layer F.SilkS)
       (effects (font (size 0.8 0.8) (thickness 0.16)))
     )
@@
     (tags "QFP 0.8")
     (attr smd)
-    (fp_text reference IC1 (at 0 -6.05 90) (layer F.SilkS)
+    (fp_text reference 328p (at -5.969 0 180) (layer F.SilkS)
       (effects (font (size 1 1) (thickness 0.15)))
     )
@@
     (descr "Through hole pin header")
     (tags "pin header")
-    (fp_text reference P3 (at -2.5781 2.8321 180) (layer F.SilkS)
+    (fp_text reference S0 (at -0.1651 7.9121 180) (layer F.SilkS)
       (effects (font (size 1 1) (thickness 0.15)))
     )
@@
     (descr "Through hole pin header")
     (tags "pin header")
-    (fp_text reference P4 (at -2.0828 2.4257 180) (layer F.SilkS)
+    (fp_text reference S1 (at -0.3048 -2.6543 180) (layer F.SilkS)
       (effects (font (size 1 1) (thickness 0.15)))
     )
@@
     (descr "Through hole pin header")
     (tags "pin header")
-    (fp_text reference P5 (at 0 -5.1) (layer F.SilkS)
+    (fp_text reference ICSP (at 1.27 7.62) (layer F.SilkS)
       (effects (font (size 1 1) (thickness 0.15)))
     )
@@
     (fp_line (start 3.81 -1.27) (end 1.27 -1.27) (layer F.SilkS) (width 0.15))
     (fp_line (start 3.81 1.27) (end 3.81 -1.27) (layer F.SilkS) (width 0.15))
-    (pad 1 thru_hole rect (at 0 0) (size 1.7272 1.7272) (drill 1.016) (layers *.Cu *.Mask F.SilkS)
+    (pad 1 thru_hole rect (at 0 0) (size 1.7272 1.7272) (drill 0.3) (layers *.Cu *.Mask F.SilkS)
       (net 22 /MISO))
-    (pad 2 thru_hole oval (at 2.54 0) (size 1.7272 1.7272) (drill 1.016) (layers *.Cu *.Mask F.SilkS)
-      (net 2 /3V3))
-    (pad 3 thru_hole oval (at 0 2.54) (size 1.7272 1.7272) (drill 1.016) (layers *.Cu *.Mask F.SilkS)
+    (pad 2 thru_hole oval (at 2.54 0) (size 1.7272 1.7272) (drill 0.3) (layers *.Cu *.Mask F.SilkS)
+      (net 2 /3V3))
+    (pad 3 thru_hole oval (at 0 2.54) (size 1.7272 1.7272) (drill 0.3) (layers *.Cu *.Mask F.SilkS)
       (net 23 /SCK))
-    (pad 4 thru_hole oval (at 2.54 2.54) (size 1.7272 1.7272) (drill 1.016) (layers *.Cu *.Mask F.SilkS)
+    (pad 4 thru_hole oval (at 2.54 2.54) (size 1.7272 1.7272) (drill 0.3) (layers *.Cu *.Mask F.SilkS)
       (net 24 /MOSI))
-    (pad 5 thru_hole oval (at 0 5.08) (size 1.7272 1.7272) (drill 1.016) (layers *.Cu *.Mask F.SilkS)
+    (pad 5 thru_hole oval (at 0 5.08) (size 1.7272 1.7272) (drill 0.3) (layers *.Cu *.Mask F.SilkS)
       (net 25 /RST))
-    (pad 6 thru_hole oval (at 2.54 5.08) (size 1.7272 1.7272) (drill 1.016) (layers *.Cu *.Mask F.SilkS)
+    (pad 6 thru_hole oval (at 2.54 5.08) (size 1.7272 1.7272) (drill 0.3) (layers *.Cu *.Mask F.SilkS)
       (net 1 /GND))
     (model Pin_Headers.3dshapes/Pin_Header_Straight_2x03.wrl
@@
     (tags "resistor 1206")
     (attr smd)
-    (fp_text reference R1 (at 0 -2.3) (layer F.SilkS)
+    (fp_text reference 4K7 (at 4.191 0) (layer F.SilkS)
       (effects (font (size 1 1) (thickness 0.15)))
     )
@@
     (descr "Through hole straight pin header, 1x02, 2.54mm pitch, single row")
     (tags "Through hole pin header THT 1x02 2.54mm single row")
-    (fp_text reference P6 (at 0 -2.39 180) (layer F.SilkS)
+    (fp_text reference 3V3 (at 0 -2.39 180) (layer F.SilkS)
       (effects (font (size 1 1) (thickness 0.15)))
     )
@@
       (effects (font (size 1 1) (thickness 0.15)) (justify mirror))
     )
-    (fp_text value CONN_01X02 (at 14 -2) (layer B.SilkS)
+    (fp_text value CR2032 (at 14 -2) (layer B.SilkS)
       (effects (font (size 1 1) (thickness 0.15)) (justify mirror))
     )
@@
     (descr "Through hole straight pin header, 1x02, 2.54mm pitch, single row")
     (tags "Through hole pin header THT 1x02 2.54mm single row")
-    (fp_text reference 3V3 (at -1.651 1.397 180) (layer F.SilkS)
+    (fp_text reference VIN (at -1.651 1.397 180) (layer F.SilkS)
       (effects (font (size 1 1) (thickness 0.15)))
     )
@@
     (tags "capacitor 1206")
     (attr smd)
-    (fp_text reference C2 (at 0 -2.3 90) (layer F.SilkS)
+    (fp_text reference 10uF (at 0.127 -1.778 90) (layer F.SilkS)
       (effects (font (size 1 1) (thickness 0.15)))
     )
@@
     (tags "resistor 1206")
     (attr smd)
-    (fp_text reference R2 (at 0 -2.3) (layer F.SilkS)
+    (fp_text reference 4K7 (at 4.191 -0.381) (layer F.SilkS)
       (effects (font (size 1 1) (thickness 0.15)))
     )
@@
     (tags "CMS SOT")
     (attr smd)
-    (fp_text reference U2 (at 0 -4.5) (layer F.SilkS)
-      (effects (font (size 1 1) (thickness 0.15)))
-    )
-    (fp_text value AP111733 (at 0 4.5) (layer F.Fab)
+    (fp_text reference 1117 (at -0.254 0 90) (layer F.SilkS)
+      (effects (font (size 1 1) (thickness 0.15)))
+    )
+    (fp_text value AP111733 (at -0.381 2.286) (layer F.Fab)
       (effects (font (size 1 1) (thickness 0.15)))
     )
@@
   (gr_line (start 131.623 51.938) (end 81.623 51.938) (angle 90) (layer Edge.Cuts) (width 0.15))
   (gr_line (start 81.623 51.938) (end 131.623 51.938) (angle 90) (layer Edge.Cuts) (width 0.15))
-  (segment (start 84.48 61.327) (end 91.454 61.327) (width 0.25) (layer F.Cu) (net 1) (status 400000))
-  (segment (start 89.2429 56.6039) (end 89.2429 54.4449) (width 0.25) (layer B.Cu) (net 1) (status 800000))
+  (segment (start 84.48 61.327) (end 91.454 61.327) (width 0.25) (layer F.Cu) (net 1))
+  (segment (start 89.2429 56.6039) (end 89.2429 54.4449) (width 0.25) (layer B.Cu) (net 1))
   (segment (start 92.71 60.071) (end 89.2429 56.6039) (width 0.25) (layer B.Cu) (net 1))
   (via (at 92.71 60.071) (size 0.6) (drill 0.4) (layers F.Cu B.Cu) (net 1))
@@
   (segment (start 100.095 72.244) (end 99.949 72.39) (width 0.25) (layer F.Cu) (net 1))
   (segment (start 99.949 72.39) (end 99.822 72.517) (width 0.25) (layer F.Cu) (net 1))
-  (segment (start 84.36 58.293) (end 83.566 58.293) (width 0.25) (layer F.Cu) (net 2) (status C00000))
-  (segment (start 83.566 58.293) (end 82.804 59.055) (width 0.25) (layer F.Cu) (net 2) (status 400000))
+  (segment (start 84.36 58.293) (end 83.566 58.293) (width 0.25) (layer F.Cu) (net 2))
+  (segment (start 83.566 58.293) (end 82.804 59.055) (width 0.25) (layer F.Cu) (net 2))
   (segment (start 82.804 59.055) (end 82.804 63.5) (width 0.25) (layer F.Cu) (net 2))
-  (segment (start 84.48 63.627) (end 82.931 63.627) (width 0.25) (layer F.Cu) (net 2) (status 400000))
+  (segment (start 84.48 63.627) (end 82.931 63.627) (width 0.25) (layer F.Cu) (net 2))
   (segment (start 82.931 63.627) (end 82.804 63.5) (width 0.25) (layer F.Cu) (net 2))
-  (segment (start 90.78 63.627) (end 84.48 63.627) (width 0.25) (layer F.Cu) (net 2) (status C00000))
+  (segment (start 90.78 63.627) (end 84.48 63.627) (width 0.25) (layer F.Cu) (net 2))
   (segment (start 100.895 70.671) (end 100.895 71.685) (width 0.25) (layer F.Cu) (net 2))
   (segment (start 100.895 71.685) (end 104.521 75.311) (width 0.25) (layer F.Cu) (net 2))
@@
   (via (at 114.554 64.135) (size 0.6) (drill 0.4) (layers F.Cu B.Cu) (net 28))
   (segment (start 117.7224 60.9666) (end 114.554 64.135) (width 0.25) (layer F.Cu) (net 28))
-  (segment (start 84.4423 75.54214) (end 83.54314 75.54214) (width 0.25) (layer F.Cu) (net 36) (status 400000))
+  (segment (start 84.4423 75.54214) (end 83.54314 75.54214) (width 0.25) (layer F.Cu) (net 36))
   (segment (start 83.54314 75.54214) (end 83.185 75.184) (width 0.25) (layer F.Cu) (net 36))
   (segment (start 83.185 69.596) (end 84.074 68.707) (width 0.25) (layer F.Cu) (net 36))
