File: domo_arduino_gradateur_puissance/domo_gradateur_puissance.kicad_pcb (KiCad board)
At the start: 2 copper layers, 100 x 100 mm, 68 parts, among them IC1 ATMEGA328-A, P1 CONN_01X01, P10 CONN_01X02, P11 5VIN, P12 ICSP, P2 CONN_01X02, P3 CONN_01X02, P4 CONN_01X02, P5 CONN_01X02, P6 CONN_01X02, P7 CONN_01X02, P8 CONN_01X02, P9 CONN_01X02, U1 LTV-814, U10 MOC3023M, U11 MOC3023M, U12 MOC3023M, U13 MOC3023M, U14 TRIAC_small, U15 TRIAC_small, U16 TRIAC_small, U17 TRIAC_small, U18 TRIAC_small, U19 TRIAC_small, U2 AP1117D33, U20 TRIAC_small, U21 TRIAC_small, U3 RFM69HW, U6 MOC3023M, U7 MOC3023M, U8 MOC3023M, U9 MOC3023M

Commit message: Ajout GERBER
Parts:
- renumbered U2 to 1117, IC1 to 328p, P11 to 5V, P1 to ANT, P12 to ICSP, U3 to RFM69HW
Connections:
- 328p pad 21: Net-(IC1-Pad21) -> GND
Routing:
- net GND: track 72.9 -> 79.7 mm
- net /SCK: track 29.1 -> 23.0 mm, vias 1 -> 0
- net /3V3: track 140.7 -> 146.4 mm
- net /IRQ: track 62.5 -> 58.1 mm
- net /C1: track 27.1 -> 25.6 mm
Other:
- board text added: "0V"
