File: domo_arduino_gradateur_puissance/domo_gradateur_puissance.sch (KiCad schematic (older format))
At the start: 68 parts, among them IC1 ATMEGA328-A, P1 CONN_01X01, P10 CONN_01X02, P11 5VIN, P12 ICSP, P2 CONN_01X02, P3 CONN_01X02, P4 CONN_01X02, P5 CONN_01X02, P6 CONN_01X02, P7 CONN_01X02, P8 CONN_01X02, P9 CONN_01X02, U1 LTV-814, U10 MOC3023M, U11 MOC3023M, U12 MOC3023M, U13 MOC3023M, U14 TRIAC_small, U15 TRIAC_small, U16 TRIAC_small, U17 TRIAC_small, U18 TRIAC_small, U19 TRIAC_small, U2 AP1117D33, U20 TRIAC_small, U21 TRIAC_small, U3 RFM69HW, U6 MOC3023M, U7 MOC3023M, U8 MOC3023M, U9 MOC3023M

Commit message: Ajout GERBER
Connections:
- wire segments 155 -> 156
Changed lines of the file:
@@
 LIBS:contrib
 LIBS:valves
-LIBS:arduino
-LIBS:ArduProMiniTKB
 LIBS:myLibrary
-LIBS:mysensors_regulators
-LIBS:mysensors_radios
 LIBS:domo_gradateur_puissance-cache
 EELAYER 25 0
@@
 	750  3000 1150 3000
 Wire Wire Line
-	1150 5300 1000 5300
-Wire Wire Line
-	1000 5300 1000 5200
+	1000 5300 1150 5300
+Wire Wire Line
+	1000 5100 1000 5300
 Wire Wire Line
 	700  5200 1150 5200
@@
 Text Label 2950 2100 0    60   ~ 0
 GND
+Wire Wire Line
+	1150 5100 1000 5100
 $EndSCHEMATC
