File: mySensors_8FilPilotes/mySensors_8FilPilotes.kicad_pcb (KiCad board)
At the start: 2 copper layers, 79 x 98 mm, 64 parts, among them P2 ANT, U10 MOC3041M, U11 MOC3041M, U12 MOC3041M, U13 MOC3041M, U14 MOC3041M, U15 MOC3041M, U16 MOC3041M, U17 MOC3041M, U18 MOC3041M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

Commit message: Ajout GERBER
Parts:
- renumbered REG to 1117, U2 to RFM69HW
Routing:
- net GND: track 47.8 -> 67.6 mm, vias 1 -> 2
