File: mySensors_FilPilote/mySensors_FilPilote_RFM69.kicad_pcb (KiCad board)
At the start: 2 copper layers, 47.5 x 49 mm, 14 parts, among them IC1 ATMEGA328-A, P1 CONN_01X03, P2 ICSP, P3 ANT, U1 MOC3041M, U2 MOC3041M, U3 AMS1117, U4 RFM69HW, U5 HLK-PM01

Commit message: correction passerelle
Routing:
- net /OPT1: track 23.0 -> 20.3 mm
