File: mySensors_2Relais/mySensors_2Relais.kicad_pcb (KiCad board)
At the start: 2 copper layers, 56 x 57 mm, 20 parts, among them IC1 ATMEGA328-A, P1 CONN_01X02, P2 ANT, P3 CONN_02X03, P4 CONN_01X03, P5 CONN_01X03, P6 CONN_01X03, Q1 PZT2222A, Q2 PZT2222A, U1 AMS1117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

Commit message: Modifications mineures
Parts:
- IN1   IN2   COM: renamed from P6; value CONN_01X03 -> (none)
- P4, P5: value CONN_01X03 -> (none)
- renumbered R1 to 390, R2 to 390, P2 to ANT, P3 to ICSP
Other:
- board text added: "AC IN"
- board text added: "C"
- board text added: "NC"
- board text added: "NO"
Changed lines of the file:
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@@
-(kicad_pcb (version 20160815) (host pcbnew no-vcs-found-7500~57~ubuntu16.04.1)
+(kicad_pcb (version 4) (host pcbnew 4.0.5-e0-6337~49~ubuntu16.04.1)
   (general
     (links 51)
     (no_connects 0)
-    (area 102.8825 55.274 178.830001 123.6765)
+    (area 102.865 55.274 178.68 123.659)
     (thickness 1.6)
-    (drawings 6)
+    (drawings 24)
     (tracks 225)
     (zones 0)
@@
       (hpglpenspeed 20)
       (hpglpendiameter 15)
+      (hpglpenoverlay 2)
       (psnegative false)
       (psa4output false)
@@
     (tags "capacitor 1206")
     (attr smd)
-    (fp_text reference C1 (at 0 -2.3 270) (layer F.SilkS)
+    (fp_text reference C1 (at 0.127 0 270) (layer F.SilkS)
       (effects (font (size 1 1) (thickness 0.15)))
     )
@@
     (tags "capacitor 1206")
     (attr smd)
-    (fp_text reference C2 (at 0 -2.3 90) (layer F.SilkS)
+    (fp_text reference C2 (at 0 0 90) (layer F.SilkS)
       (effects (font (size 1 1) (thickness 0.15)))
     )
@@
     (descr "Through hole straight pin header, 1x01, 2.54mm pitch, single row")
     (tags "Through hole pin header THT 1x01 2.54mm single row")
-    (fp_text reference P2 (at 0 -2.39) (layer F.SilkS)
+    (fp_text reference ANT (at 0 -2.39) (layer F.SilkS)
       (effects (font (size 1 1) (thickness 0.15)))
     )
@@
     (descr "Through hole straight pin header, 2x03, 2.54mm pitch, double rows")
     (tags "Through hole pin header THT 2x03 2.54mm double row")
-    (fp_text reference P3 (at 1.27 -2.39 180) (layer F.SilkS)
+    (fp_text reference ICSP (at 1.27 -2.39 180) (layer F.SilkS)
       (effects (font (size 1 1) (thickness 0.15)))
     )
@@
       (effects (font (size 1 1) (thickness 0.15)))
     )
-    (fp_text value CONN_01X03 (at 5.08 5.08 90) (layer F.Fab)
+    (fp_text value "" (at 5.08 5.08 90) (layer F.Fab)
       (effects (font (size 1 1) (thickness 0.15)))
     )
@@
       (effects (font (size 1 1) (thickness 0.15)))
     )
-    (fp_text value CONN_01X03 (at 5.08 5.08 270) (layer F.Fab)
+    (fp_text value "" (at 5.08 5.08 270) (layer F.Fab)
       (effects (font (size 1 1) (thickness 0.15)))
     )
@@
     (descr "Bornier d'alimentation 3 pins")
     (tags DEV)
-    (fp_text reference P6 (at 5.05 -4.65 90) (layer F.SilkS)
-      (effects (font (size 1 1) (thickness 0.15)))
-    )
-    (fp_text value CONN_01X03 (at 5.08 5.08 90) (layer F.Fab)
+    (fp_text reference "IN1   IN2   COM" (at 5.05 -4.65 90) (layer F.SilkS)
+      (effects (font (size 1 1) (thickness 0.15)))
+    )
+    (fp_text value "" (at 5.08 5.08 90) (layer F.Fab)
       (effects (font (size 1 1) (thickness 0.15)))
     )
@@
     (tags SOT-23)
     (attr smd)
-    (fp_text reference Q1 (at 0 -2.5) (layer F.SilkS)
+    (fp_text reference Q1 (at 1.8415 -1.27) (layer F.SilkS)
       (effects (font (size 1 1) (thickness 0.15)))
     )
@@
     (tags SOT-23)
     (attr smd)
-    (fp_text reference Q2 (at 0 -2.5) (layer F.SilkS)
+    (fp_text reference Q2 (at 1.778 -1.397) (layer F.SilkS)
       (effects (font (size 1 1) (thickness 0.15)))
     )
@@
     (tags "resistor 1206")
     (attr smd)
-    (fp_text reference R1 (at 0 -2.3 180) (layer F.SilkS)
+    (fp_text reference 390 (at 0 -0.0635 180) (layer F.SilkS)
       (effects (font (size 1 1) (thickness 0.15)))
     )
@@
     (tags "resistor 1206")
     (attr smd)
-    (fp_text reference R2 (at 0 -2.3) (layer F.SilkS)
+    (fp_text reference 390 (at 0 0.127) (layer F.SilkS)
       (effects (font (size 1 1) (thickness 0.15)))
     )
@@
   (module MyLibrary:SRD_Relay_TypeC (layer F.Cu)
     (at 142.875 113.284)
-    (fp_text reference RLY1 (at 0 9) (layer F.SilkS)
+    (fp_text reference RLY1 (at 0 5.08) (layer F.SilkS)
       (effects (font (size 1 1) (thickness 0.15)))
     )
@@
   (module MyLibrary:SRD_Relay_TypeC (layer F.Cu)
     (at 123.19 113.284 180)
-    (fp_text reference RLY2 (at 0 9 180) (layer F.SilkS)
+    (fp_text reference RLY2 (at 0 -5.08 180) (layer F.SilkS)
       (effects (font (size 1 1) (thickness 0.15)))
     )
@@
     (tags "CMS SOT")
     (attr smd)
-    (fp_text reference U1 (at 0 -4.5 270) (layer F.SilkS)
+    (fp_text reference U1 (at 0 -0.127 270) (layer F.SilkS)
       (effects (font (size 1 1) (thickness 0.15)))
     )
@@
     (tags SOD-123)
     (attr smd)
-    (fp_text reference D1 (at 0 -2) (layer F.SilkS)
+    (fp_text reference D1 (at 0 0) (layer F.SilkS)
       (effects (font (size 1 1) (thickness 0.15)))
     )
@@
     (tags SOD-123)
     (attr smd)
-    (fp_text reference D2 (at 0 -2 270) (layer F.SilkS)
+    (fp_text reference D2 (at 0 1.651 270) (layer F.SilkS)
       (effects (font (size 1 1) (thickness 0.15)))
     )
@@
     )
   )
-  (dimension 57 (width 0.3) (layer F.SilkS)
-    (gr_text "57,000 mm" (at 172.18 92.474 270) (layer F.SilkS)
-      (effects (font (size 1.5 1.5) (thickness 0.3)))
-    )
-    (feature1 (pts (xy 160.83 120.974) (xy 173.53 120.974)))
-    (feature2 (pts (xy 160.83 63.974) (xy 173.53 63.974)))
-    (crossbar (pts (xy 170.83 63.974) (xy 170.83 120.974)))
-    (arrow1a (pts (xy 170.83 120.974) (xy 170.243579 119.847496)))
-    (arrow1b (pts (xy 170.83 120.974) (xy 171.416421 119.847496)))
-    (arrow2a (pts (xy 170.83 63.974) (xy 170.243579 65.100504)))
-    (arrow2b (pts (xy 170.83 63.974) (xy 171.416421 65.100504)))
-  )
-  (dimension 56 (width 0.3) (layer F.SilkS)
-    (gr_text "56,000 mm" (at 132.83 56.624) (layer F.SilkS)
-      (effects (font (size 1.5 1.5) (thickness 0.3)))
-    )
-    (feature1 (pts (xy 160.83 63.974) (xy 160.83 55.274)))
-    (feature2 (pts (xy 104.83 63.974) (xy 104.83 55.274)))
-    (crossbar (pts (xy 104.83 57.974) (xy 160.83 57.974)))
-    (arrow1a (pts (xy 160.83 57.974) (xy 159.703496 58.560421)))
-    (arrow1b (pts (xy 160.83 57.974) (xy 159.703496 57.387579)))
-    (arrow2a (pts (xy 104.83 57.974) (xy 105.956504 58.560421)))
-    (arrow2b (pts (xy 104.83 57.974) (xy 105.956504 57.387579)))
-  )
+  (gr_text "AC\nIN" (at 110.363 81.407) (layer F.SilkS)
+    (effects (font (size 1.5 1.5) (thickness 0.3)))
+  )
+  (gr_text "C\n" (at 153.924 112.395) (layer B.SilkS)
+    (effects (font (size 1.5 1.5) (thickness 0.3)) (justify mirror))
+  )
+  (gr_text "C\n" (at 112.268 112.268) (layer B.SilkS)
+    (effects (font (size 1.5 1.5) (thickness 0.3)) (justify mirror))
+  )
+  (gr_text NO (at 112.395 117.475) (layer B.SilkS)
+    (effects (font (size 1.5 1.5) (thickness 0.3)) (justify mirror))
+  )
+  (gr_text NO (at 153.162 107.188) (layer B.SilkS)
+    (effects (font (size 1.5 1.5) (thickness 0.3)) (justify mirror))
+  )
+  (gr_text NC (at 153.035 117.348) (layer B.SilkS)
+    (effects (font (size 1.5 1.5) (thickness 0.3)) (justify mirror))
+  )
+  (gr_text NC (at 113.03 107.061) (layer B.SilkS)
+    (effects (font (size 1.5 1.5) (thickness 0.3)) (justify mirror))
+  )
+  (gr_line (start 113.284 113.284) (end 109.728 113.284) (angle 90) (layer B.SilkS) (width 0.2))
+  (gr_line (start 113.411 113.284) (end 113.284 113.284) (angle 90) (layer B.SilkS) (width 0.2))
+  (gr_line (start 116.586 110.109) (end 113.411 113.284) (angle 90) (layer B.SilkS) (width 0.2))
+  (gr_line (start 116.713 118.364) (end 116.713 115.951) (angle 90) (layer B.SilkS) (width 0.2))
+  (gr_line (start 109.347 118.364) (end 116.713 118.364) (angle 90) (layer B.SilkS) (width 0.2))
+  (gr_line (start 116.586 108.204) (end 116.586 109.982) (angle 90) (layer B.SilkS) (width 0.2))
+  (gr_line (start 110.109 108.204) (end 116.586 108.204) (angle 90) (layer B.SilkS) (width 0.2))
+  (gr_line (start 148.336 108.204) (end 155.448 108.204) (angle 90) (layer B.SilkS) (width 0.2))
+  (gr_line (start 148.336 110.109) (end 148.336 108.204) (angle 90) (layer B.SilkS) (width 0.2))
+  (gr_line (start 148.336 118.364) (end 148.336 116.205) (angle 90) (layer B.SilkS) (width 0.2))
+  (gr_line (start 151.003 113.411) (end 148.082 116.332) (angle 90) (layer B.SilkS) (width 0.2))
+  (gr_line (start 155.194 118.364) (end 148.209 118.364) (angle 90) (layer B.SilkS) (width 0.2))
+  (gr_line (start 155.448 113.411) (end 151.003 113.411) (angle 90) (layer B.SilkS) (width 0.2))
   (gr_line (start 104.83 63.974) (end 104.83 120.974) (angle 90) (layer Edge.Cuts) (width 0.15))
   (gr_line (start 160.83 120.974) (end 160.83 63.974) (angle 90) (layer Edge.Cuts) (width 0.15))
