File: mySensors_2Relais/mySensors_2Relais.sch (KiCad schematic (older format))
At the start: 20 parts, among them IC1 ATMEGA328-A, P1 CONN_01X02, P2 ANT, P3 CONN_02X03, P4 CONN_01X03, P5 CONN_01X03, P6 CONN_01X03, Q1 PZT2222A, Q2 PZT2222A, U1 AMS1117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

Commit message: Modifications mineures
Parts:
- P1: value CONN_01X02 -> 220V
- Q1, Q2: value PZT2222A -> MBT2222
- R1, R2: value R -> 390
Changed lines of the file:
@@
 LIBS:contrib
 LIBS:valves
+LIBS:mysensors_radios
+LIBS:mysensors_regulators
 LIBS:myLibrary
 LIBS:relay_spdt
 LIBS:uln-udn
 LIBS:mySensors_2Relais-cache
-EELAYER 26 0
+EELAYER 25 0
 EELAYER END
 $Descr A4 11693 8268
@@
 P 5200 5250
 F 0 "Q1" H 5391 5341 50  0000 L CNN
-F 1 "PZT2222A" H 5391 5250 50  0000 L CNN
+F 1 "MBT2222" H 5391 5250 50  0000 L CNN
 F 2 "TO_SOT_Packages_SMD:SOT-23" H 5391 5159 50  0000 L CIN
 F 3 "" H 5200 5250 50  0000 L CNN
@@
 P 4800 5250
 F 0 "R1" V 4593 5250 50  0000 C CNN
-F 1 "R" V 4684 5250 50  0000 C CNN
+F 1 "390" V 4684 5250 50  0000 C CNN
 F 2 "Resistors_SMD:R_1206_HandSoldering" V 4730 5250 50  0001 C CNN
 F 3 "" H 4800 5250 50  0000 C CNN
@@
 P 5200 6050
 F 0 "Q2" H 5391 6141 50  0000 L CNN
-F 1 "PZT2222A" H 5391 6050 50  0000 L CNN
+F 1 "MBT2222" H 5391 6050 50  0000 L CNN
 F 2 "TO_SOT_Packages_SMD:SOT-23" H 5391 5959 50  0000 L CIN
 F 3 "" H 5200 6050 50  0000 L CNN
@@
 P 4800 6050
 F 0 "R2" V 4593 6050 50  0000 C CNN
-F 1 "R" V 4684 6050 50  0000 C CNN
+F 1 "390" V 4684 6050 50  0000 C CNN
 F 2 "Resistors_SMD:R_1206_HandSoldering" V 4730 6050 50  0001 C CNN
 F 3 "" H 4800 6050 50  0000 C CNN
@@
 P 700 1100
 F 0 "P1" H 778 1141 50  0000 L CNN
-F 1 "CONN_01X02" H 778 1050 50  0000 L CNN
+F 1 "220V" H 778 1050 50  0000 L CNN
 F 2 "Connectors:bornier2" H 700 1100 50  0001 C CNN
 F 3 "" H 700 1100 50  0000 C CNN
