File: mySensors_8Relais/mySensors_8Relais.sch (KiCad schematic (older format))
At the start: 33 parts, among them IC1 ATMEGA328-A, IC2 ULN2803A, P1 5VIN, P10 CONN_01X03, P11 CONN_01X03, P2 ANT, P3 CONN_02X03, P4 CONN_01X03, P5 CONN_01X03, P6 CONN_01X03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

Commit message: Terminé le circuit 8 Relais
Parts:
- U2: footprint Mysensors_Radio:RFM69HW_SMD_Handsoldering -> mysensors-radio:RFM69HW_SMD_Handsoldering
Changed lines of the file:
@@
 LIBS:contrib
 LIBS:valves
-LIBS:mysensors_radios
-LIBS:mysensors_regulators
-LIBS:myLibrary
 LIBS:relay_spdt
 LIBS:uln-udn
 LIBS:mySensors_8Relais-cache
-EELAYER 25 0
+EELAYER 26 0
 EELAYER END
 $Descr A4 11693 8268
@@
 F 0 "U2" H 2000 5600 40  0000 C CNN
 F 1 "RFM69HW" H 2600 4600 40  0000 C CNN
-F 2 "Mysensors_Radio:RFM69HW_SMD_Handsoldering" H 2350 5350 30  0001 C CIN
+F 2 "mysensors-radio:RFM69HW_SMD_Handsoldering" H 2350 5350 30  0001 C CIN
 F 3 "" H 2350 5350 60  0000 C CNN
 	1    2350 5350
@@
 IRQ
 Text Label 5800 5250 0    60   ~ 0
+S0
+Text Label 5800 5350 0    60   ~ 0
+S1
+Text Label 5800 5450 0    60   ~ 0
+S2
+Text Label 5800 5550 0    60   ~ 0
+S3
+Text Label 5800 5650 0    60   ~ 0
+S4
+Text Label 5800 5750 0    60   ~ 0
+S5
+Text Label 5800 5850 0    60   ~ 0
+S6
+Text Label 5800 5950 0    60   ~ 0
 S7
-Text Label 5800 5350 0    60   ~ 0
-S6
-Text Label 5800 5450 0    60   ~ 0
-S5
-Text Label 5800 5550 0    60   ~ 0
-S4
-Text Label 5800 5650 0    60   ~ 0
-S3
-Text Label 5800 5750 0    60   ~ 0
-S2
-Text Label 5800 5850 0    60   ~ 0
-S1
-Text Label 5800 5950 0    60   ~ 0
-S0
 Wire Wire Line
 	1000 1050 1100 1050
@@
 F 3 "" H 8900 800 50  0000 C CNN
 	1    8900 800
-	1    0    0    -1
+	1    0    0    1
 $EndComp
 $Comp
@@
 F 3 "" H 8900 1400 50  0000 C CNN
 	1    8900 1400
-	1    0    0    -1
+	1    0    0    1
 $EndComp
 $Comp
@@
 F 3 "" H 8900 2000 50  0000 C CNN
 	1    8900 2000
-	1    0    0    -1
+	1    0    0    1
 $EndComp
 $Comp
@@
 F 3 "" H 8900 2600 50  0000 C CNN
 	1    8900 2600
-	1    0    0    -1
+	1    0    0    1
 $EndComp
 $Comp
@@
 F 3 "" H 8900 3200 50  0000 C CNN
 	1    8900 3200
-	1    0    0    -1
+	1    0    0    1
 $EndComp
 $Comp
@@
 F 3 "" H 8900 3800 50  0000 C CNN
 	1    8900 3800
-	1    0    0    -1
+	1    0    0    1
 $EndComp
 $Comp
@@
 F 3 "" H 8900 4400 50  0000 C CNN
 	1    8900 4400
-	1    0    0    -1
+	1    0    0    1
 $EndComp
 $Comp
@@
 F 3 "" H 8900 5000 50  0000 C CNN
 	1    8900 5000
-	1    0    0    -1
+	1    0    0    1
 $EndComp
 $Comp
@@
 	4300 5250 4650 5250
 Text Label 4350 5250 0    60   ~ 0
+SL0
+Text Label 4350 5350 0    60   ~ 0
+SL1
+Text Label 4350 5450 0    60   ~ 0
+SL2
+Text Label 4350 5550 0    60   ~ 0
+SL3
+Text Label 4350 5650 0    60   ~ 0
+SL4
+Text Label 4350 5750 0    60   ~ 0
+SL5
+Text Label 4350 5850 0    60   ~ 0
+SL6
+Text Label 4350 5950 0    60   ~ 0
 SL7
-Text Label 4350 5350 0    60   ~ 0
-SL6
-Text Label 4350 5450 0    60   ~ 0
-SL5
-Text Label 4350 5550 0    60   ~ 0
-SL4
-Text Label 4350 5650 0    60   ~ 0
-SL3
-Text Label 4350 5750 0    60   ~ 0
-SL2
-Text Label 4350 5850 0    60   ~ 0
-SL1
-Text Label 4350 5950 0    60   ~ 0
-SL0
 Wire Wire Line
 	3600 2850 3300 2850

Commit message: Modifications mineures
Parts:
- removed D1, D2, D3, D4, D5, D6, D7, D8: D, Diodes_SMD:SOD-123, symbol D
Connections:
- wire segments 145 -> 146
Changed lines of the file:
@@
 LIBS:contrib
 LIBS:valves
+LIBS:mysensors_radios
+LIBS:mysensors_regulators
+LIBS:myLibrary
 LIBS:relay_spdt
 LIBS:uln-udn
 LIBS:mySensors_8Relais-cache
-EELAYER 26 0
+EELAYER 25 0
 EELAYER END
 $Descr A4 11693 8268
@@
 Text Label 7550 4950 0    60   ~ 0
 VCC
-$Comp
-L D D1
-U 1 1 58768BBC
-P 7350 900
-F 0 "D1" H 7350 1000 50  0000 C CNN
-F 1 "D" H 7350 800 50  0000 C CNN
-F 2 "Diodes_SMD:SOD-123" H 7350 900 50  0001 C CNN
-F 3 "" H 7350 900 50  0000 C CNN
-	1    7350 900
-	0    1    1    0
-$EndComp
-$Comp
-L D D2
-U 1 1 58768C8C
-P 7350 1500
-F 0 "D2" H 7350 1600 50  0000 C CNN
-F 1 "D" H 7350 1400 50  0000 C CNN
-F 2 "Diodes_SMD:SOD-123" H 7350 1500 50  0001 C CNN
-F 3 "" H 7350 1500 50  0000 C CNN
-	1    7350 1500
-	0    1    1    0
-$EndComp
-$Comp
-L D D3
-U 1 1 58768D34
-P 7350 2100
-F 0 "D3" H 7350 2200 50  0000 C CNN
-F 1 "D" H 7350 2000 50  0000 C CNN
-F 2 "Diodes_SMD:SOD-123" H 7350 2100 50  0001 C CNN
-F 3 "" H 7350 2100 50  0000 C CNN
-	1    7350 2100
-	0    1    1    0
-$EndComp
-$Comp
-L D D4
-U 1 1 58768E5D
-P 7350 2700
-F 0 "D4" H 7350 2800 50  0000 C CNN
-F 1 "D" H 7350 2600 50  0000 C CNN
-F 2 "Diodes_SMD:SOD-123" H 7350 2700 50  0001 C CNN
-F 3 "" H 7350 2700 50  0000 C CNN
-	1    7350 2700
-	0    1    1    0
-$EndComp
-$Comp
-L D D5
-U 1 1 58768F13
-P 7350 3300
-F 0 "D5" H 7350 3400 50  0000 C CNN
-F 1 "D" H 7350 3200 50  0000 C CNN
-F 2 "Diodes_SMD:SOD-123" H 7350 3300 50  0001 C CNN
-F 3 "" H 7350 3300 50  0000 C CNN
-	1    7350 3300
-	0    1    1    0
-$EndComp
-$Comp
-L D D6
-U 1 1 5876905D
-P 7350 3900
-F 0 "D6" H 7350 4000 50  0000 C CNN
-F 1 "D" H 7350 3800 50  0000 C CNN
-F 2 "Diodes_SMD:SOD-123" H 7350 3900 50  0001 C CNN
-F 3 "" H 7350 3900 50  0000 C CNN
-	1    7350 3900
-	0    1    1    0
-$EndComp
-$Comp
-L D D7
-U 1 1 58769113
-P 7350 4500
-F 0 "D7" H 7350 4600 50  0000 C CNN
-F 1 "D" H 7350 4400 50  0000 C CNN
-F 2 "Diodes_SMD:SOD-123" H 7350 4500 50  0001 C CNN
-F 3 "" H 7350 4500 50  0000 C CNN
-	1    7350 4500
-	0    1    1    0
-$EndComp
-$Comp
-L D D8
-U 1 1 587691CE
-P 7350 5100
-F 0 "D8" H 7350 5200 50  0000 C CNN
-F 1 "D" H 7350 5000 50  0000 C CNN
-F 2 "Diodes_SMD:SOD-123" H 7350 5100 50  0001 C CNN
-F 3 "" H 7350 5100 50  0000 C CNN
-	1    7350 5100
-	0    1    1    0
-$EndComp
 Wire Wire Line
 	1000 950  1200 950
@@
 Text Label 3400 3700 0    60   ~ 0
 SL0
+Wire Wire Line
+	5650 6050 6000 6050
+Text Label 5800 6050 0    60   ~ 0
+VCC
 $EndSCHEMATC
