File: mySensors_8RelaisReed/mySensors_8RelaisReed.kicad_pcb (KiCad board)
At the start: 2 copper layers, 81.3 x 59.7 mm, 33 parts, among them IC1 ATMEGA328-A, P1 5VIN, P10 CONN_01X02, P11 CONN_01X02, P2 ANT, P3 CONN_02X03, P4 CONN_01X02, P5 CONN_01X02, P6 CONN_01X02, P7 CONN_01X02, P8 CONN_01X02, P9 CONN_01X02, U1 AMS1117, U2 RFM69HW, U3 74HC595

Commit message: Ajout GERBER
Parts:
- +5V   0V: renamed from P1
- moved +5V   0V 0.64 mm to (143.5, 114.3)
- renumbered U1 to 1117, IC1 to 328p, U3 to 74HC595, P2 to ANT, P3 to ICSP, U2 to RFM69HW, P4 to S1, P5 to S2, P6 to S3, P7 to S4, P8 to S5, P9 to S6, P10 to S7, P11 to S8

Commit message: Rename of  domo_arduino_gradateur_puissance to  MySensors_8Dimmers  project. Added first version of MySensors_4Blinds firmware (for 8 Reed Relays board) Added pull-up resistor on radio module for 8 reed relays board.
Parts:
- added R9: 10k, Resistors_SMD:R_1206_HandSoldering, F.Cu at (213.6, 105.7)
- P1: renamed from +5V   0V
- renumbered 328p to IC1, S7 to P10, S8 to P11, ANT to P2, ICSP to P3, S1 to P4, S2 to P5, S3 to P6, S4 to P7, S5 to P8, S6 to P9, 1117 to U1, RFM69HW to U2, 74HC595 to U3
Routing:
- net /CS: track 32.6 -> 56.3 mm
- net /3V3: track 102.8 -> 105.8 mm
Changed lines of the file:
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@@
-(kicad_pcb (version 4) (host pcbnew 4.0.5-e0-6337~49~ubuntu16.04.1)
+(kicad_pcb (version 20170123) (host pcbnew no-vcs-found-7560~57~ubuntu16.04.1)
   (general
-    (links 81)
+    (links 83)
     (no_connects 0)
-    (area 137.155 63.495 220.285001 125.825)
+    (area 138.354999 65.964999 219.785001 125.805001)
     (thickness 1.6)
     (drawings 4)
-    (tracks 233)
+    (tracks 239)
     (zones 0)
-    (modules 33)
+    (modules 34)
     (nets 64)
   )
@@
       (hpglpenspeed 20)
       (hpglpendiameter 15)
-      (hpglpenoverlay 2)
       (psnegative false)
       (psa4output false)
@@
     (tags "QFP 0.8")
     (attr smd)
-    (fp_text reference 328p (at 0 -6.05) (layer F.SilkS)
+    (fp_text reference IC1 (at 0 -6.05) (layer F.SilkS)
       (effects (font (size 1 1) (thickness 0.15)))
     )
@@
     (descr "Bornier d'alimentation 2 pins")
     (tags DEV)
-    (fp_text reference "+5V   0V" (at 0 -5.08 270) (layer F.SilkS)
+    (fp_text reference P1 (at 0 -5.08 270) (layer F.SilkS)
       (effects (font (size 1 1) (thickness 0.15)))
     )
@@
     (descr "Through hole straight pin header, 1x01, 2.54mm pitch, single row")
     (tags "Through hole pin header THT 1x01 2.54mm single row")
-    (fp_text reference ANT (at 0 -2.39) (layer F.SilkS)
+    (fp_text reference P2 (at 0 -2.39) (layer F.SilkS)
       (effects (font (size 1 1) (thickness 0.15)))
     )
@@
     (descr "Through hole straight pin header, 2x03, 2.54mm pitch, double rows")
     (tags "Through hole pin header THT 2x03 2.54mm double row")
-    (fp_text reference ICSP (at 1.27 -2.39 180) (layer F.SilkS)
+    (fp_text reference P3 (at 1.27 -2.39 180) (layer F.SilkS)
       (effects (font (size 1 1) (thickness 0.15)))
     )
@@
     (descr "Bornier d'alimentation 2 pins")
     (tags DEV)
-    (fp_text reference S1 (at -0.127 -4.572 180) (layer F.SilkS)
+    (fp_text reference P4 (at -0.127 -4.572 180) (layer F.SilkS)
       (effects (font (size 1 1) (thickness 0.15)))
     )
@@
     (descr "Bornier d'alimentation 2 pins")
     (tags DEV)
-    (fp_text reference S2 (at 0 -4.572 180) (layer F.SilkS)
+    (fp_text reference P5 (at 0 -4.572 180) (layer F.SilkS)
       (effects (font (size 1 1) (thickness 0.15)))
     )
@@
     (descr "Bornier d'alimentation 2 pins")
     (tags DEV)
-    (fp_text reference S3 (at 0 -4.445 180) (layer F.SilkS)
+    (fp_text reference P6 (at 0 -4.445 180) (layer F.SilkS)
       (effects (font (size 1 1) (thickness 0.15)))
     )
@@
     (descr "Bornier d'alimentation 2 pins")
     (tags DEV)
-    (fp_text reference S4 (at 0 -4.572 180) (layer F.SilkS)
+    (fp_text reference P7 (at 0 -4.572 180) (layer F.SilkS)
       (effects (font (size 1 1) (thickness 0.15)))
     )
@@
     (descr "Bornier d'alimentation 2 pins")
     (tags DEV)
-    (fp_text reference S5 (at 0 -4.572 180) (layer F.SilkS)
+    (fp_text reference P8 (at 0 -4.572 180) (layer F.SilkS)
       (effects (font (size 1 1) (thickness 0.15)))
     )
@@
     (descr "Bornier d'alimentation 2 pins")
     (tags DEV)
-    (fp_text reference S6 (at 0 -4.572 180) (layer F.SilkS)
+    (fp_text reference P9 (at 0 -4.572 180) (layer F.SilkS)
       (effects (font (size 1 1) (thickness 0.15)))
     )
@@
     (descr "Bornier d'alimentation 2 pins")
     (tags DEV)
-    (fp_text reference S7 (at 0 -4.572 180) (layer F.SilkS)
+    (fp_text reference P10 (at 0 -4.572 180) (layer F.SilkS)
       (effects (font (size 1 1) (thickness 0.15)))
     )
@@
     (descr "Bornier d'alimentation 2 pins")
     (tags DEV)
-    (fp_text reference S8 (at 0 -4.572 180) (layer F.SilkS)
+    (fp_text reference P11 (at 0 -4.572 180) (layer F.SilkS)
       (effects (font (size 1 1) (thickness 0.15)))
     )
@@
     (tags "CMS SOT")
     (attr smd)
-    (fp_text reference 1117 (at 0 -4.5) (layer F.SilkS)
+    (fp_text reference U1 (at 0 -4.5) (layer F.SilkS)
       (effects (font (size 1 1) (thickness 0.15)))
     )
@@
     (descr RFM69HW)
     (tags "RFM69HW, RF69")
-    (fp_text reference RFM69HW (at 0.254 -1.778 180) (layer F.SilkS)
+    (fp_text reference U2 (at 0.254 -1.778 180) (layer F.SilkS)
       (effects (font (size 0.8 0.8) (thickness 0.16)))
     )
@@
     (tags "CMS SOJ")
     (attr smd)
-    (fp_text reference 74HC595 (at 0.127 -1.27 180) (layer F.SilkS)
+    (fp_text reference U3 (at 0.127 -1.27 180) (layer F.SilkS)
       (effects (font (size 1 1) (thickness 0.15)))
     )
@@
     )
   )
+  (module Resistors_SMD:R_1206_HandSoldering (layer F.Cu)
+    (at 213.614 105.664 180)
+    (descr "Resistor SMD 1206, hand soldering")
+    (tags "resistor 1206")
+    (attr smd)
+    (fp_text reference R9 (at 0 -1.85 180) (layer F.SilkS)
+      (effects (font (size 1 1) (thickness 0.15)))
+    )
+    (fp_text value 10k (at 0 1.9 180) (layer F.Fab)
+      (effects (font (size 1 1) (thickness 0.15)))
+    )
+    (fp_line (start 3.25 1.1) (end -3.25 1.1) (layer F.CrtYd) (width 0.05))
+    (fp_line (start 3.25 1.1) (end 3.25 -1.11) (layer F.CrtYd) (width 0.05))
+    (fp_line (start -3.25 -1.11) (end -3.25 1.1) (layer F.CrtYd) (width 0.05))
+    (fp_line (start -3.25 -1.11) (end 3.25 -1.11) (layer F.CrtYd) (width 0.05))
+    (fp_line (start -1 -1.07) (end 1 -1.07) (layer F.SilkS) (width 0.12))
+    (fp_line (start 1 1.07) (end -1 1.07) (layer F.SilkS) (width 0.12))
+    (fp_line (start -1.6 -0.8) (end 1.6 -0.8) (layer F.Fab) (width 0.1))
+    (fp_line (start 1.6 -0.8) (end 1.6 0.8) (layer F.Fab) (width 0.1))
+    (fp_line (start 1.6 0.8) (end -1.6 0.8) (layer F.Fab) (width 0.1))
+    (fp_line (start -1.6 0.8) (end -1.6 -0.8) (layer F.Fab) (width 0.1))
+    (fp_text user %R (at 0 -1.85 180) (layer F.Fab)
+      (effects (font (size 1 1) (thickness 0.15)))
+    )
+    (pad 2 smd rect (at 2 0 180) (size 2 1.7) (layers F.Cu F.Paste F.Mask)
+      (net 12 /CS))
+    (pad 1 smd rect (at -2 0 180) (size 2 1.7) (layers F.Cu F.Paste F.Mask)
+      (net 4 /3V3))
+    (model Resistors_SMD.3dshapes/R_1206.wrl
+      (at (xyz 0 0 0))
+      (scale (xyz 1 1 1))
+      (rotate (xyz 0 0 0))
+    )
+  )
   (gr_line (start 138.43 125.73) (end 138.43 66.04) (angle 90) (layer Edge.Cuts) (width 0.15))
   (gr_line (start 219.71 125.73) (end 138.43 125.73) (angle 90) (layer Edge.Cuts) (width 0.15))
@@
   (segment (start 166.44 116.275) (end 163.39 116.275) (width 0.25) (layer F.Cu) (net 3))
   (segment (start 167.24 117.075) (end 166.44 116.275) (width 0.25) (layer F.Cu) (net 3))
+  (segment (start 215.395 108.555) (end 215.395 105.883) (width 0.25) (layer F.Cu) (net 4) (status C00000))
+  (segment (start 215.395 105.883) (end 215.614 105.664) (width 0.25) (layer F.Cu) (net 4) (status C00000))
   (segment (start 181.483 123.8351) (end 162.6971 123.8351) (width 0.25) (layer F.Cu) (net 4))
   (segment (start 162.6971 123.8351) (end 161.671 122.809) (width 0.25) (layer F.Cu) (net 4))
@@
   (segment (start 153.1153 109.0056) (end 151.765 107.6553) (width 0.25) (layer F.Cu) (net 4))
   (segment (start 153.1153 114.3) (end 153.1153 109.0056) (width 0.25) (layer F.Cu) (net 4))
+  (segment (start 195.695 120.555) (end 199.485 120.555) (width 0.25) (layer F.Cu) (net 12) (status 400000))
+  (segment (start 209.423 107.855) (end 211.614 105.664) (width 0.25) (layer F.Cu) (net 12) (status 800000))
+  (segment (start 209.423 110.617) (end 209.423 107.855) (width 0.25) (layer F.Cu) (net 12))
+  (segment (start 199.485 120.555) (end 209.423 110.617) (width 0.25) (layer F.Cu) (net 12))
   (segment (start 168.84 121.725) (end 168.84 119.818) (width 0.25) (layer F.Cu) (net 12))
   (segment (start 173.609 124.587) (end 178.181 124.587) (width 0.25) (layer B.Cu) (net 12))
