File: mySensors_8RelaisReed/mySensors_8RelaisReed.sch (KiCad schematic (older format))
At the start: 33 parts, among them IC1 ATMEGA328-A, P1 5VIN, P10 CONN_01X02, P11 CONN_01X02, P2 ANT, P3 CONN_02X03, P4 CONN_01X02, P5 CONN_01X02, P6 CONN_01X02, P7 CONN_01X02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

Commit message: Rename of  domo_arduino_gradateur_puissance to  MySensors_8Dimmers  project. Added first version of MySensors_4Blinds firmware (for 8 Reed Relays board) Added pull-up resistor on radio module for 8 reed relays board.
Parts:
- added R9: 10k, Resistors_SMD:R_1206_HandSoldering, symbol R
Connections:
- wire segments 88 -> 91
Changed lines of the file:
@@
 LIBS:contrib
 LIBS:valves
-LIBS:mysensors_radios
-LIBS:mysensors_regulators
-LIBS:myLibrary
-LIBS:mySensors_16Outputs-cache
-EELAYER 25 0
+LIBS:mySensors_8RelaisReed-cache
+EELAYER 26 0
 EELAYER END
 $Descr A4 11693 8268
@@
 	2350 5000 2700 5000
 Wire Wire Line
-	3300 2200 3600 2200
+	3300 2200 3750 2200
 Wire Wire Line
 	1400 2000 1000 2000
@@
 Text Label 2550 6300 0    60   ~ 0
 GND
+$Comp
+L R R9
+U 1 1 58B2DB4E
+P 3750 2000
+F 0 "R9" H 3820 2046 50  0000 L CNN
+F 1 "10k" H 3820 1955 50  0000 L CNN
+F 2 "Resistors_SMD:R_1206_HandSoldering" V -120 50  50  0001 C CNN
+F 3 "" H -50 50  50  0001 C CNN
+	1    3750 2000
+	1    0    0    -1
+$EndComp
+Wire Wire Line
+	3750 2200 3750 2150
+Wire Wire Line
+	3750 1850 3750 1800
+Wire Wire Line
+	3750 1800 4000 1800
+Text Label 3800 1800 0    60   ~ 0
+3V3
 $EndSCHEMATC
