File: MultiUse_Battery_RFM69HCW/MultiUse_Battery_RFM69HCW.sch (KiCad schematic (older format))
At the start: 13 parts, among them IC1 ATMEGA328P-AU, P1 CONN_01X02, P2 CONN_01X01, P3 CONN_01X03, P4 CONN_01X03, P5 CONN_02X03, P6 CONN_01X02, U2 AP111733, U3 RFM69HCW

Commit message: Update to MultiUse_Battery_RFM69HCW (schematic + firmware) WIP of mySensors_Teleinfo
Parts:
- removed R5: 0, Resistors_SMD:R_1206_HandSoldering, symbol R
- added C2: 10uF, Capacitors_SMD:C_1206_HandSoldering, symbol C
- added JP1: Jumper, MyLibrary:Jump, symbol Jumper
- S1: renamed from P3; footprint Pin_Headers:Pin_Header_Straight_1x03 -> Pin_Headers:Pin_Header_Straight_1x03_Pitch2.54mm
- S2: renamed from P4; footprint Pin_Headers:Pin_Header_Straight_1x03 -> Pin_Headers:Pin_Header_Straight_1x03_Pitch2.54mm
- renumbered P6 to 3VIN1, P2 to ANT1, C4 to C1, P5 to ICSP1, U3 to U1
Connections:
- wire segments 57 -> 58
Other:
- note removed: "Si utilisation pile : \n- Souder 0R sur R5"
Changed lines of the file:
@@
 LIBS:contrib
 LIBS:valves
-LIBS:mysensors_radios
-LIBS:myLibrary
 LIBS:MultiUse_Battery_RFM69HCW-cache
-EELAYER 26 0
+EELAYER 25 0
 EELAYER END
 $Descr A4 11693 8268
@@
 $EndComp
 $Comp
-L CONN_01X03 P4
+L CONN_01X03 S2
 U 1 1 587A3CDC
 P 9150 4900
-F 0 "P4" H 9228 4941 50  0000 L CNN
+F 0 "S2" H 9228 4941 50  0000 L CNN
 F 1 "CONN_01X03" H 9228 4850 50  0000 L CNN
-F 2 "Pin_Headers:Pin_Header_Straight_1x03" H 9150 4900 50  0001 C CNN
+F 2 "Pin_Headers:Pin_Header_Straight_1x03_Pitch2.54mm" H 9150 4900 50  0001 C CNN
 F 3 "" H 9150 4900 50  0000 C CNN
 	1    9150 4900
@@
 $EndComp
 $Comp
-L CONN_01X03 P3
+L CONN_01X03 S1
 U 1 1 587A3D32
 P 9050 3850
-F 0 "P3" H 9128 3891 50  0000 L CNN
+F 0 "S1" H 9128 3891 50  0000 L CNN
 F 1 "CONN_01X03" H 9128 3800 50  0000 L CNN
-F 2 "Pin_Headers:Pin_Header_Straight_1x03" H 9050 3850 50  0001 C CNN
+F 2 "Pin_Headers:Pin_Header_Straight_1x03_Pitch2.54mm" H 9050 3850 50  0001 C CNN
 F 3 "" H 9050 3850 50  0000 C CNN
 	1    9050 3850
@@
 GND
 $Comp
-L CONN_01X01 P2
+L CONN_01X01 ANT1
 U 1 1 587A904D
 P 4700 5850
-F 0 "P2" H 4619 5625 50  0000 C CNN
+F 0 "ANT1" H 4619 5625 50  0000 C CNN
 F 1 "CONN_01X01" H 4619 5716 50  0000 C CNN
 F 2 "Pin_Headers:Pin_Header_Straight_1x01" H 4700 5850 50  0001 C CNN
@@
 PC1
 $Comp
-L CONN_02X03 P5
+L CONN_02X03 ICSP1
 U 1 1 587A7114
 P 9000 2650
-F 0 "P5" H 9000 2850 50  0000 C CNN
+F 0 "ICSP1" H 9000 2850 50  0000 C CNN
 F 1 "CONN_02X03" H 9000 2450 50  0000 C CNN
 F 2 "Pin_Headers:Pin_Header_Straight_2x03" H 9000 1450 50  0001 C CNN
@@
 3V3
 $Comp
-L RFM69HCW U3
+L RFM69HCW U1
 U 1 1 58890FD8
 P 5650 6000
-F 0 "U3" H 5650 6505 40  0000 C CNN
+F 0 "U1" H 5650 6505 40  0000 C CNN
 F 1 "RFM69HCW" H 5650 6429 40  0000 C CNN
 F 2 "MyLibrary:RFM69HCW_HandSolder" H 5650 6450 30  0001 C CIN
@@
 Connection ~ 5650 6900
 $Comp
-L C C4
+L C C1
 U 1 1 58890DEC
 P 2550 2750
-F 0 "C4" H 2665 2796 50  0000 L CNN
+F 0 "C1" H 2665 2796 50  0000 L CNN
 F 1 "100nF" H 2665 2705 50  0000 L CNN
 F 2 "Capacitors_SMD:C_1206_HandSoldering" H 2588 2600 50  0001 C CNN
@@
 Text Label 2300 2900 0    60   ~ 0
 GND
-Text Notes 6000 950  0    60   ~ 0
-Si utilisation pile : \n- Souder 0R sur R5
 Wire Wire Line
 	1800 1200 2100 1200
@@
 Text Label 1850 1300 0    60   ~ 0
 GND
-$Comp
-L R R5
-U 1 1 58892177
-P 6350 1150
-F 0 "R5" V 6450 1100 50  0000 L CNN
-F 1 "0" V 6250 1100 50  0000 L CNN
-F 2 "Resistors_SMD:R_1206_HandSoldering" V 6280 1150 50  0001 C CNN
-F 3 "" H 6350 1150 50  0001 C CNN
-	1    6350 1150
-	0    1    1    0
-$EndComp
-Wire Wire Line
-	6200 1150 5950 1150
-Wire Wire Line
-	5950 1150 5950 1650
 Connection ~ 5950 1650
-Wire Wire Line
-	6500 1150 6750 1150
-Wire Wire Line
-	6750 1150 6750 1650
 Connection ~ 6750 1650
 $Comp
-L CONN_01X02 P6
+L CONN_01X02 3VIN1
 U 1 1 588929E7
 P 1600 1950
-F 0 "P6" H 1519 1675 50  0000 C CNN
+F 0 "3VIN1" H 1519 1675 50  0000 C CNN
 F 1 "CONN_01X02" H 1519 1766 50  0000 C CNN
 F 2 "Pin_Headers:Pin_Header_Straight_1x02_Pitch2.54mm" H 1600 1950 50  0001 C CNN
@@
 	2850 3200 2900 3200
 Connection ~ 2850 2900
+$Comp
+L C C2
+U 1 1 5889A70B
+P 6750 1800
+F 0 "C2" H 6865 1846 50  0000 L CNN
+F 1 "10uF" H 6865 1755 50  0000 L CNN
+F 2 "Capacitors_SMD:C_1206_HandSoldering" H 6788 1650 50  0001 C CNN
+F 3 "" H 6750 1800 50  0000 C CNN
+	1    6750 1800
+	1    0    0    -1
+$EndComp
+Wire Wire Line
+	6750 1950 6750 2050
+Connection ~ 6750 2050
+$Comp
+L Jumper JP1
+U 1 1 5889C53F
+P 6350 1200
+F 0 "JP1" H 6350 1350 50  0000 C CNN
+F 1 "Jumper" H 6350 1120 50  0000 C CNN
+F 2 "MyLibrary:Jump" H 6350 1450 50  0000 C CNN
+F 3 "" H 6350 1200 50  0000 C CNN
+	1    6350 1200
+	1    0    0    -1
+$EndComp
+Wire Wire Line
+	6050 1200 5950 1200
+Wire Wire Line
+	5950 1200 5950 1650
+Wire Wire Line
+	6650 1200 6750 1200
+Wire Wire Line
+	6750 1200 6750 1650
 $EndSCHEMATC
