File: MySensors_Gateway/MySensors_Gateway.kicad_pcb (KiCad board)
At the start: 2 copper layers, 12 parts, among them P1 CONN_01X01, U1 AP111733, U2 arduino_mini, U3 RFM69HW

Commit message: correction passerelle
Parts:
- added P2: CONN_01X02, Pin_Headers:Pin_Header_Straight_1x02_Pitch2.54mm, F.Cu at (150.4, 125.0)
- added P3: CONN_01X02, Pin_Headers:Pin_Header_Straight_1x02_Pitch2.54mm, F.Cu at (159.8, 125.0)
- added U4: 74HC245, Housings_SOIC:SOIC-20W_7.5x12.8mm_Pitch1.27mm, B.Cu at (176.8, 108.6)
- moved P1 38.4 mm to (186.8, 102.1)
- moved R3 35.2 mm to (144.8, 117.9), turned to 90 degrees
- moved R2 30.9 mm to (139.6, 117.9), turned to 90 degrees
- moved R1 27.4 mm to (134.5, 117.9), turned to 90 degrees
- moved U1 25.0 mm to (154.2, 118.2), turned to 180 degrees
- moved D1 24.8 mm to (134.4, 125.3), turned to 90 degrees
- moved C2 23.6 mm to (166.2, 120.5), turned to 270 degrees
- moved D2 22.2 mm to (139.6, 125.3), turned to 90 degrees
- moved D3 20.7 mm to (144.8, 125.3), turned to 90 degrees
- moved C1 17.7 mm to (162.4, 116.0), turned to 270 degrees
- moved U3 2.72 mm to (170.2, 116.7)
Connections:
- net /3V3 renamed VCC
- U3 pad 12: /SCK -> /SCK3
- U3 pad 13: /MISO -> /MISO3
- U3 pad 14: /MOSI -> /MOSI3
- U3 pad 15: /CS -> /CS3
- U3 pad 2: /IRQ -> /IRQ3
Routing:
- net VCC: track 0.00 -> 76.2 mm
- net /MOSI: track 0.00 -> 59.1 mm
- net /SCK: track 0.00 -> 56.5 mm
- net /CS: track 0.00 -> 53.5 mm
- net /MISO: track 0.00 -> 53.2 mm
- net GND: track 0.00 -> 32.0 mm
- net /VUSB: track 0.00 -> 26.2 mm
- net /IRQ: track 0.00 -> 26.2 mm
- net /MISO3: track 0.00 -> 15.4 mm, vias 0 -> 1
- net /IRQ3: track 0.00 -> 11.0 mm, vias 0 -> 1
- net /CS3: track 0.00 -> 9.73 mm, vias 0 -> 1
- net /MOSI3: track 0.00 -> 9.05 mm, vias 0 -> 1
- net Net-(P1-Pad1): track 0.00 -> 7.56 mm
- net /SCK3: track 0.00 -> 6.21 mm, vias 0 -> 1
- net /LED_ERR: track 0.00 -> 5.89 mm
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- added copper zone on B.Cu, net GND
- added copper zone on F.Cu, net GND
Other:
- board outline added: 64 x 34 mm

Commit message: Update to MultiUse_Battery_RFM69HCW (schematic + firmware) WIP of mySensors_Teleinfo
Connections:
- U2 pad 10: Net-(U2-Pad10) -> (no net)
- U2 pad 11: Net-(U2-Pad11) -> (no net)
- U2 pad 13: Net-(U2-Pad13) -> (no net)
- U2 pad 15: Net-(U2-Pad15) -> (no net)
- U2 pad 16: Net-(U2-Pad16) -> (no net)
- U2 pad 17: Net-(U2-Pad17) -> (no net)
- U2 pad 18: Net-(U2-Pad18) -> (no net)
- U2 pad 2: Net-(U2-Pad2) -> (no net)
- U2 pad 21: Net-(U2-Pad21) -> (no net)
- U2 pad 22: Net-(U2-Pad22) -> (no net)
- U2 pad 23: Net-(U2-Pad23) -> (no net)
- U2 pad 24: Net-(U2-Pad24) -> (no net)
- U2 pad 25: Net-(U2-Pad25) -> (no net)
- U2 pad 26: Net-(U2-Pad26) -> (no net)
- U2 pad 27: Net-(U2-Pad27) -> (no net)
- U2 pad 3: Net-(U2-Pad3) -> (no net)
- U2 pad 7: Net-(U2-Pad7) -> (no net)
- U2 pad 8: Net-(U2-Pad8) -> (no net)
- U2 pad 9: Net-(U2-Pad9) -> (no net)
- U3 pad 1: Net-(U3-Pad1) -> (no net)
- U3 pad 16: Net-(U3-Pad16) -> (no net)
- U3 pad 2: /IRQ3 -> /IRQ
- U3 pad 3: Net-(U3-Pad3) -> (no net)
- U3 pad 4: Net-(U3-Pad4) -> (no net)
- U3 pad 5: Net-(U3-Pad5) -> (no net)
- U3 pad 6: Net-(U3-Pad6) -> (no net)
- U3 pad 7: Net-(U3-Pad7) -> (no net)
- U4 pad 11: Net-(U4-Pad11) -> (no net)
- U4 pad 12: Net-(U4-Pad12) -> (no net)
- U4 pad 13: Net-(U4-Pad13) -> (no net)
- U4 pad 14: /IRQ -> (no net)
- U4 pad 6: /IRQ3 -> (no net)
- U4 pad 7: Net-(U4-Pad7) -> (no net)
- U4 pad 8: Net-(U4-Pad8) -> (no net)
- U4 pad 9: Net-(U4-Pad9) -> (no net)
Routing:
- net /IRQ3: track 11.0 -> 0.00 mm, vias 1 -> 0
- net /IRQ: track 26.2 -> 27.9 mm
