File: MySensors_Gateway/MySensors_Gateway.sch (KiCad schematic (older format))
At the start: 12 parts, among them P1 CONN_01X01, U1 AP111733, U2 arduino_mini, U3 RFM69HW

Commit message: correction passerelle
Parts:
- added P2, P3: CONN_01X02, Pin_Headers:Pin_Header_Straight_1x02_Pitch2.54mm, symbol CONN_01X02
- added U4: 74HC245, Housings_SOIC:SOIC-20W_7.5x12.8mm_Pitch1.27mm, symbol 74HC245
Connections:
- net labels added: CS3, IRQ3, MISO3, MOSI3, SCK3, VCC
- wire segments 40 -> 61
Other:
- moved on the sheet: C1, C2, D1, D2, D3, R1, R2, R3, U1

Commit message: Update to MultiUse_Battery_RFM69HCW (schematic + firmware) WIP of mySensors_Teleinfo
Connections:
- net labels removed: IRQ3
- wire segments 61 -> 59
Changed lines of the file:
@@
 3V3
 Text Label 8100 4500 0    60   ~ 0
-IRQ3
+IRQ
 Text Label 7800 5450 0    60   ~ 0
 GND
@@
 VCC
 Wire Wire Line
-	6900 3000 6400 3000
-Text Label 6450 3000 0    60   ~ 0
-IRQ3
-Wire Wire Line
-	8300 3000 8700 3000
-Text Label 8400 3000 0    60   ~ 0
-IRQ
-Wire Wire Line
 	6900 3500 6400 3500
